Commit message: Signed-off-by: Andrea Patrizi <andreapatrizi1b6e6@gmail.com>

File: centauro_urdf/urdf/parts/head.urdf.xacro (robot description, xacro)
@@ -138,6 +138,6 @@
       <origin xyz="${d435_cam_mount_from_center_offset} ${-d435_cam_depth_py} 0" rpy="${PI/2} 0 ${PI/2}"/>
         <geometry>
-          <!-- <box size="${d435_cam_width} ${d435_cam_height} ${d435_cam_depth}"/> -->
-          <mesh filename="${MESH_PATH}/realsense/d435.dae"/>
+          <box size="${d435_cam_width} ${d435_cam_height} ${d435_cam_depth}"/>
+          <!-- <mesh filename="${MESH_PATH}/realsense/d435.dae"/> -->
         </geometry>
         <material name="${d435_head_name}_aluminum"/>
