Commit message: restored usage of mesh for wheels, since IsaacSim uses meshes anyway for cylinders

File: centauro_urdf/urdf/parts/wheel23.urdf.xacro (robot description, xacro)
@@ -53,11 +53,11 @@
             <collision>
                 <origin xyz="0 0 0" rpy="0 0 0" />
+                <!-- <geometry>
+					<cylinder radius="${wheel23_radius}" length="${wheel23_depth}"/>
+				</geometry> -->
                 <geometry>
-					<cylinder radius="${wheel23_radius}" length="${wheel23_depth}"/>
-				</geometry>
-                <!-- <geometry>
                     <mesh filename="${MESH_PATH}/v2/collision/mesh_wheel23.stl"
                         scale="0.001 0.001 ${mirror*0.001}" />
-                </geometry> -->
+                </geometry>
                 <material name="black" />
             </collision>

Commit message: using donut wheels for collision

File: centauro_urdf/urdf/parts/wheel23.urdf.xacro (robot description, xacro)
@@ -18,5 +18,5 @@
                 <material name="dark_grey" />
             </visual>
-            <collision>
+            <!-- <collision>
                 <origin xyz="0.0 0.0 0.0" rpy="0.0 0.0 0.0" />
                 <geometry>
@@ -25,5 +25,5 @@
                         scale="0.001 ${mirror*0.001} 0.001" />
                 </geometry>
-            </collision>
+            </collision> -->
         </link>
         <joint name="j_wheel_${leg_num}" type="continuous">
@@ -53,11 +53,11 @@
             <collision>
                 <origin xyz="0 0 0" rpy="0 0 0" />
+                <!-- <geometry>
+					<cylinder radius="${wheel23_radius}" length="${wheel23_depth}"/>
+				</geometry> -->
                 <geometry>
-					<cylinder radius="${wheel23_radius}" length="${wheel23_depth}"/>
-				</geometry>
-                <!-- <geometry>
-                    <mesh filename="${MESH_PATH}/v2/collision/mesh_wheel23.stl"
+                    <mesh filename="${MESH_PATH}/v2/collision/wheel23_donut.stl"
                         scale="0.001 0.001 ${mirror*0.001}" />
-                </geometry> -->
+                </geometry>
                 <material name="black" />
             </collision>

Commit message: added donut wheel collisions

File: centauro_urdf/urdf/parts/wheel23.urdf.xacro (robot description, xacro)
@@ -18,5 +18,5 @@
                 <material name="dark_grey" />
             </visual>
-            <collision>
+            <!-- <collision>
                 <origin xyz="0.0 0.0 0.0" rpy="0.0 0.0 0.0" />
                 <geometry>
@@ -25,5 +25,5 @@
                         scale="0.001 ${mirror*0.001} 0.001" />
                 </geometry>
-            </collision>
+            </collision> -->
         </link>
         <joint name="j_wheel_${leg_num}" type="continuous">
@@ -57,5 +57,5 @@
 				</geometry> -->
                 <geometry>
-                    <mesh filename="${MESH_PATH}/v2/collision/mesh_wheel23.stl"
+                    <mesh filename="${MESH_PATH}/v2/collision/wheel23_donut.stl"
                         scale="0.001 0.001 ${mirror*0.001}" />
                 </geometry>

Commit message: reverted to using cylinder for wheel collision

File: centauro_urdf/urdf/parts/wheel23.urdf.xacro (robot description, xacro)
@@ -53,11 +53,11 @@
             <collision>
                 <origin xyz="0 0 0" rpy="0 0 0" />
+                <geometry>
+					<cylinder radius="${wheel23_radius}" length="${wheel23_depth}"/>
+				</geometry>
                 <!-- <geometry>
-					<cylinder radius="${wheel23_radius}" length="${wheel23_depth}"/>
-				</geometry> -->
-                <geometry>
                     <mesh filename="${MESH_PATH}/v2/collision/wheel23_donut.stl"
                         scale="0.001 0.001 ${mirror*0.001}" />
-                </geometry>
+                </geometry> -->
                 <material name="black" />
             </collision>
