Commit message: new homing

File: centauro_srdf/srdf/centauro.srdf.xacro (robot description, xacro)
@@ -71,5 +71,5 @@
     </group>
     <!-- Homing posture -->
-    <group_state name="home" group="chains">
+    <!-- <group_state name="home" group="chains">
         <joint name="hip_yaw_1" value="-0.746874"/>
         <joint name="hip_pitch_1" value="-1.25409"/>
@@ -117,4 +117,52 @@
             <joint name="dagana_2_claw_joint" value="0"/>
         </xacro:if>
+    </group_state> -->
+    <!-- Balanced weight homing -->
+    <group_state name="home" group="chains">
+        <joint name="hip_yaw_1" value="-0.5"/>
+        <joint name="hip_pitch_1" value="-1.37"/>
+        <joint name="knee_pitch_1" value="-1.34"/>
+        <joint name="ankle_pitch_1" value="-0.03"/>
+        <joint name="ankle_yaw_1" value="0.75"/>
+        <joint name="hip_yaw_2" value="0.5"/>
+        <joint name="hip_pitch_2" value="1.37"/>
+        <joint name="knee_pitch_2" value="1.34"/>
+        <joint name="ankle_pitch_2" value="-0.03"/>
+        <joint name="ankle_yaw_2" value="-0.75"/>
+        <joint name="hip_yaw_3" value="1.28"/>
+        <joint name="hip_pitch_3" value="1.29"/>
+        <joint name="knee_pitch_3" value="1.71"/>
+        <joint name="ankle_pitch_3" value="0.43"/>
+        <joint name="ankle_yaw_3" value="-0.75"/>
+        <joint name="hip_yaw_4" value="-1.28"/>
+        <joint name="hip_pitch_4" value="-1.29"/>
+        <joint name="knee_pitch_4" value="-1.71"/>
+        <joint name="ankle_pitch_4" value="-0.43"/>
+        <joint name="ankle_yaw_4" value="0.75"/>
+        <joint name="torso_yaw" value="3.56617e-13"/>
+        <joint name="velodyne_joint" value="0"/>
+        <joint name="d435_head_joint" value="0"/>
+        <joint name="j_arm1_1" value="0.520149"/>
+        <joint name="j_arm1_2" value="0.320865"/>
+        <joint name="j_arm1_3" value="0.274669"/>
+        <joint name="j_arm1_4" value="-2.23604"/>
+        <joint name="j_arm1_5" value="0.0500815"/>
+        <joint name="j_arm1_6" value="-0.781461"/>
+        <joint name="j_arm2_1" value="0.520149"/>
+        <joint name="j_arm2_2" value="-0.320865"/>
+        <joint name="j_arm2_3" value="-0.274669"/>
+        <joint name="j_arm2_4" value="-2.23604"/>
+        <joint name="j_arm2_5" value="-0.0500815"/>
+        <joint name="j_arm2_6" value="-0.781461"/>
+        <joint name="j_wheel_1" value="0.0"/>
+        <joint name="j_wheel_2" value="0.0"/>
+        <joint name="j_wheel_3" value="0.0"/>
+        <joint name="j_wheel_4" value="0.0"/>
+        <xacro:if value="${END_EFFECTOR_LEFT == 'dagana'}">
+            <joint name="dagana_1_claw_joint" value="0"/>
+        </xacro:if>
+        <xacro:if value="${END_EFFECTOR_RIGHT == 'dagana'}">
+            <joint name="dagana_2_claw_joint" value="0"/>
+        </xacro:if>
     </group_state>
 </robot>

Commit message: Signed-off-by: AndrePatri <andreapatrizi97@gmail.com>

File: centauro_srdf/srdf/centauro.srdf.xacro (robot description, xacro)
@@ -124,20 +124,20 @@
         <joint name="knee_pitch_1" value="-1.34"/>
         <joint name="ankle_pitch_1" value="-0.03"/>
-        <joint name="ankle_yaw_1" value="0.75"/>
+        <joint name="ankle_yaw_1" value="0.6"/>
         <joint name="hip_yaw_2" value="0.5"/>
         <joint name="hip_pitch_2" value="1.37"/>
         <joint name="knee_pitch_2" value="1.34"/>
         <joint name="ankle_pitch_2" value="-0.03"/>
-        <joint name="ankle_yaw_2" value="-0.75"/>
+        <joint name="ankle_yaw_2" value="-0.6"/>
         <joint name="hip_yaw_3" value="1.28"/>
         <joint name="hip_pitch_3" value="1.29"/>
         <joint name="knee_pitch_3" value="1.71"/>
         <joint name="ankle_pitch_3" value="0.43"/>
-        <joint name="ankle_yaw_3" value="-0.75"/>
+        <joint name="ankle_yaw_3" value="-1.3"/>
         <joint name="hip_yaw_4" value="-1.28"/>
         <joint name="hip_pitch_4" value="-1.29"/>
         <joint name="knee_pitch_4" value="-1.71"/>
         <joint name="ankle_pitch_4" value="-0.43"/>
-        <joint name="ankle_yaw_4" value="0.75"/>
+        <joint name="ankle_yaw_4" value="1.3"/>
         <joint name="torso_yaw" value="3.56617e-13"/>
         <joint name="velodyne_joint" value="0"/>

Commit message: fixed mismatch between ros1 and ros2 branches (added missing new homing)

File: centauro_srdf/srdf/centauro.srdf.xacro (robot description, xacro)
@@ -71,5 +71,5 @@
     </group>
     <!-- Homing posture -->
-    <group_state name="home" group="chains">
+    <!-- <group_state name="home" group="chains">
         <joint name="hip_yaw_1" value="-0.746874"/>
         <joint name="hip_pitch_1" value="-1.25409"/>
@@ -117,4 +117,52 @@
             <joint name="dagana_2_claw_joint" value="0"/>
         </xacro:if>
+    </group_state> -->
+    <!-- Balanced weight homing -->
+    <group_state name="home" group="chains">
+        <joint name="hip_yaw_1" value="-0.5"/>
+        <joint name="hip_pitch_1" value="-1.37"/>
+        <joint name="knee_pitch_1" value="-1.34"/>
+        <joint name="ankle_pitch_1" value="-0.03"/>
+        <joint name="ankle_yaw_1" value="0.6"/>
+        <joint name="hip_yaw_2" value="0.5"/>
+        <joint name="hip_pitch_2" value="1.37"/>
+        <joint name="knee_pitch_2" value="1.34"/>
+        <joint name="ankle_pitch_2" value="-0.03"/>
+        <joint name="ankle_yaw_2" value="-0.6"/>
+        <joint name="hip_yaw_3" value="1.28"/>
+        <joint name="hip_pitch_3" value="1.29"/>
+        <joint name="knee_pitch_3" value="1.71"/>
+        <joint name="ankle_pitch_3" value="0.43"/>
+        <joint name="ankle_yaw_3" value="-1.3"/>
+        <joint name="hip_yaw_4" value="-1.28"/>
+        <joint name="hip_pitch_4" value="-1.29"/>
+        <joint name="knee_pitch_4" value="-1.71"/>
+        <joint name="ankle_pitch_4" value="-0.43"/>
+        <joint name="ankle_yaw_4" value="1.3"/>
+        <joint name="torso_yaw" value="3.56617e-13"/>
+        <joint name="velodyne_joint" value="0"/>
+        <joint name="d435_head_joint" value="0"/>
+        <joint name="j_arm1_1" value="0.520149"/>
+        <joint name="j_arm1_2" value="0.320865"/>
+        <joint name="j_arm1_3" value="0.274669"/>
+        <joint name="j_arm1_4" value="-2.23604"/>
+        <joint name="j_arm1_5" value="0.0500815"/>
+        <joint name="j_arm1_6" value="-0.781461"/>
+        <joint name="j_arm2_1" value="0.520149"/>
+        <joint name="j_arm2_2" value="-0.320865"/>
+        <joint name="j_arm2_3" value="-0.274669"/>
+        <joint name="j_arm2_4" value="-2.23604"/>
+        <joint name="j_arm2_5" value="-0.0500815"/>
+        <joint name="j_arm2_6" value="-0.781461"/>
+        <joint name="j_wheel_1" value="0.0"/>
+        <joint name="j_wheel_2" value="0.0"/>
+        <joint name="j_wheel_3" value="0.0"/>
+        <joint name="j_wheel_4" value="0.0"/>
+        <xacro:if value="${END_EFFECTOR_LEFT == 'dagana'}">
+            <joint name="dagana_1_claw_joint" value="0"/>
+        </xacro:if>
+        <xacro:if value="${END_EFFECTOR_RIGHT == 'dagana'}">
+            <joint name="dagana_2_claw_joint" value="0"/>
+        </xacro:if>
     </group_state>
 </robot>

File: centauro_urdf/urdf/parts/head.urdf.xacro (robot description, xacro)
@@ -138,6 +138,6 @@
       <origin xyz="${d435_cam_mount_from_center_offset} ${-d435_cam_depth_py} 0" rpy="${PI/2} 0 ${PI/2}"/>
         <geometry>
-          <!-- <box size="${d435_cam_width} ${d435_cam_height} ${d435_cam_depth}"/> -->
-          <mesh filename="${MESH_PATH}/realsense/d435.dae"/>
+          <box size="${d435_cam_width} ${d435_cam_height} ${d435_cam_depth}"/>
+          <!-- <mesh filename="${MESH_PATH}/realsense/d435.dae"/> -->
         </geometry>
         <material name="${d435_head_name}_aluminum"/>
