Commit message: removed typo in xacr

File: centauro_urdf/urdf/centauro.urdf.xacro (robot description, xacro)
@@ -23,7 +23,4 @@
     <xacro:property name="MESH_PATH" value="package://centauro_urdf/meshes" />
 </xacro:unless>
-<xacro:macro name="example_macro">
-  <example_element message="${MESH_PATH}" />
-</xacro:macro>
 <!-- configuration -->
 <xacro:arg name="config" default="${ROOT}/urdf/config/centauro.urdf.xacro"/>
